File: Eagle/PhasedArrayTransmittor/PhasedArrayTransmittor.brd (EAGLE design)
At the start: 100 x 80 mm, 18 parts, among them IC1 OP400P, IC2 LM555D

Commit message: Add files via upload
Parts:
- removed C1: 0.1u, rcl:C0603K
- removed C2: 1000p, rcl:C0603K
- removed C3: (no value), rcl:C0603K
- removed R1: 10k, rcl:RTRIM74W
- removed R2, R4: 10k, rcl:R0603
- removed R3: 1.5k, rcl:R0603
- removed R5: 22k, rcl:R0603
- removed R6, R7: 1, rcl:R0603
- removed T1, T2, T3, T4: (no value), transistor:SOT23-BEC
- added CPASS, CT5: 0.1u, rcl:C0603K
- added CPASST: 0.1u, rcl:C025-024X044
- added CSENS: (no value), rcl:C0603K
- added CT6: 1000p, rcl:C0603K
- added RAMP1, RT72: 10k, rcl:R0603
- added RAMP2: 22k, rcl:R0603
- added RAMPD, RAMPU: 1, rcl:R0603
- added RT7: 10k, rcl:RTRIM74W
- added RT73: 1.5k, rcl:R0603
- added TNPN1, TNPN2, TPNP1, TPNP2: (no value), transistor:SOT23-BEC
- moved JP2 170.9 mm to (81.0, 50.0), turned to 270 degrees
- moved JP1 107.9 mm to (8.00, 74.0)
- moved IC1 78.5 mm to (43.9, 47.6), turned to 180 degrees
- moved IC2 59.5 mm to (21.5, 61.2), turned to 90 degrees
Connections:
- net +5V/1: now also CPASST.1, RT73.2; no longer R3.2
- net +9V: now also CPASS.1, TNPN2.C; no longer T1.C
- net DGND: now also CPASS.2, CPASST.2, CT5.2, CT6.2, RAMP1.1, TPNP2.C; no longer C1.2, C2.2, R4.1, T4.C
- net N$1: now also CT5.1; no longer C1.1
- net N$10: now also RAMPD.1, TPNP1.B, TPNP2.E; no longer R7.1, T3.B, T4.E
- net N$13: now also RAMPU.2, TNPN1.B, TNPN2.E; no longer R6.2, T1.E, T2.B
- net N$14: now also CSENS.1, RAMP2.2, RAMPD.2, RAMPU.1, TNPN1.E, TPNP1.E; no longer C3.1, R5.2, R6.1, R7.2, T2.E, T3.E
- net N$16: now also CSENS.2; no longer C3.2
- net N$3: now also RT7.3, RT72.1; no longer R1.3, R2.1
- net N$4: now also RAMP1.2, RAMP2.1; no longer R4.2, R5.1
- net N$5: now also RT72.2, RT73.1; no longer R2.2, R3.1
- net N$7: now also TNPN1.C, TNPN2.B, TPNP1.C, TPNP2.B; no longer T1.B, T2.C, T3.C, T4.B
- net N$8: now also CT6.1, RT7.1, RT7.2; no longer C2.1, R1.1, R1.2
Routing:
- net N$14: track 0.00 -> 23.5 mm
- net N$7: track 0.00 -> 13.2 mm
- net N$13: track 0.00 -> 11.2 mm, vias 0 -> 2
- net N$10: track 0.00 -> 7.66 mm
- net N$16: track 0.00 -> 3.43 mm
- net N$4: track 0.00 -> 3.00 mm
- net DGND: track 0.00 -> 0.51 mm

Commit message: Add files via upload
Parts:
- CT5, CT6: device rcl:C0603K -> rcl:C025-024X044
- moved JP1 13.2 mm to (21.0, 76.0), turned to 180 degrees
- moved CT6 7.81 mm to (22.0, 67.0), turned to 90 degrees
- moved CT5 2.24 mm to (19.0, 67.0), turned to 90 degrees
Routing:
- net N$8: track 0.00 -> 19.7 mm
- net N$5: track 0.00 -> 8.73 mm
- net +5V/1: track 0.00 -> 8.22 mm
- net DGND: track 0.51 -> 7.07 mm
- net N$3: track 0.00 -> 2.67 mm
- net N$2: track 0.00 -> 2.65 mm
Changed lines of the file:
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@@
 <attribute name="VALUE" x="23.395" y="65.157" size="1.27" layer="27" rot="R180"/>
-</element>
-<element name="CT5" library="rcl" library_urn="urn:adsk.eagle:library:334" package="C0603K" package3d_urn="urn:adsk.eagle:package:23680/2" value="0.1u" x="21" y="66" smashed="yes">
-<attribute name="NAME" x="20.2" y="66.65" size="1.016" layer="25"/>
-<attribute name="POPULARITY" value="30" x="21" y="66" size="1.778" layer="27" display="off"/>
-<attribute name="SPICEPREFIX" value="C" x="21" y="66" size="1.778" layer="27" display="off"/>
-<attribute name="VALUE" x="20.2" y="64.35" size="1.016" layer="27"/>
 </element>
 <element name="RT7" library="rcl" library_urn="urn:adsk.eagle:library:334" package="RTRIM74W" package3d_urn="urn:adsk.eagle:package:23745/1" value="10k" x="14" y="63" smashed="yes" rot="MR180">
@@
 <attribute name="VALUE" x="15.365" y="53.095" size="1.27" layer="27"/>
 </element>
-<element name="JP1" library="pinhead" library_urn="urn:adsk.eagle:library:325" package="1X02" package3d_urn="urn:adsk.eagle:package:22435/2" value="" x="8" y="74" smashed="yes">
-<attribute name="NAME" x="5.3838" y="75.8288" size="1.27" layer="25" ratio="10"/>
-<attribute name="POPULARITY" value="98" x="8" y="74" size="1.778" layer="27" display="off"/>
-<attribute name="VALUE" x="5.46" y="70.825" size="1.27" layer="27"/>
-</element>
-<element name="CT6" library="rcl" library_urn="urn:adsk.eagle:library:334" package="C0603K" package3d_urn="urn:adsk.eagle:package:23680/2" value="1000p" x="28" y="62" smashed="yes" rot="R180">
-<attribute name="NAME" x="28.8" y="61.35" size="1.016" layer="25" rot="R180"/>
-<attribute name="POPULARITY" value="30" x="28" y="62" size="1.778" layer="27" rot="R180" display="off"/>
-<attribute name="SPICEPREFIX" value="C" x="28" y="62" size="1.778" layer="27" rot="R180" display="off"/>
-<attribute name="VALUE" x="28.8" y="63.65" size="1.016" layer="27" rot="R180"/>
+<element name="JP1" library="pinhead" library_urn="urn:adsk.eagle:library:325" package="1X02" package3d_urn="urn:adsk.eagle:package:22435/2" value="" x="21" y="76" smashed="yes" rot="R180">
+<attribute name="NAME" x="23.6162" y="74.1712" size="1.27" layer="25" ratio="10" rot="R180"/>
+<attribute name="POPULARITY" value="98" x="21" y="76" size="1.778" layer="27" rot="R180" display="off"/>
+<attribute name="VALUE" x="23.54" y="79.175" size="1.27" layer="27" rot="R180"/>
 </element>
 <element name="RAMP1" library="rcl" library_urn="urn:adsk.eagle:library:334" package="R0603" package3d_urn="urn:adsk.eagle:package:23555/3" value="10k" x="60" y="52" smashed="yes" rot="R180">
@@
 <attribute name="VALUE" x="19.222" y="53.333" size="1.27" layer="27" ratio="10"/>
 </element>
+<element name="CT5" library="rcl" library_urn="urn:adsk.eagle:library:334" package="C025-024X044" package3d_urn="urn:adsk.eagle:package:23630/1" value="0.1u" x="19" y="67" smashed="yes" rot="R90">
+<attribute name="NAME" x="17.603" y="65.222" size="1.27" layer="25" ratio="10" rot="R90"/>
+<attribute name="POPULARITY" value="56" x="19" y="67" size="1.778" layer="27" rot="R90" display="off"/>
+<attribute name="SPICEPREFIX" value="C" x="19" y="67" size="1.778" layer="27" rot="R90" display="off"/>
+<attribute name="VALUE" x="21.667" y="65.222" size="1.27" layer="27" ratio="10" rot="R90"/>
+</element>
+<element name="CT6" library="rcl" library_urn="urn:adsk.eagle:library:334" package="C025-024X044" package3d_urn="urn:adsk.eagle:package:23630/1" value="1000p" x="22" y="67" smashed="yes" rot="R90">
+<attribute name="NAME" x="20.603" y="65.222" size="1.27" layer="25" ratio="10" rot="R90"/>
+<attribute name="POPULARITY" value="56" x="22" y="67" size="1.778" layer="27" rot="R90" display="off"/>
+<attribute name="SPICEPREFIX" value="C" x="22" y="67" size="1.778" layer="27" rot="R90" display="off"/>
+<attribute name="VALUE" x="24.667" y="65.222" size="1.27" layer="27" ratio="10" rot="R90"/>
+</element>
 </elements>
 <signals>
 <signal name="DGND" class="1">
 <contactref element="IC2" pad="1"/>
-<contactref element="CT5" pad="2"/>
-<contactref element="CT6" pad="2"/>
 <contactref element="RAMP1" pad="1"/>
 <contactref element="IC1" pad="11"/>
@@
 <contactref element="JP2" pad="2"/>
 <contactref element="CPASS" pad="2"/>
-<wire x1="67.9" y1="54" x2="67.9" y2="53.48684375" width="0.9144" layer="1"/>
 <contactref element="CPASST" pad="2"/>
-<wire x1="67.9" y1="53.48684375" x2="81" y2="48.73" width="0" layer="19" extent="1-1"/>
-<wire x1="60.85" y1="52" x2="67.9" y2="53.48684375" width="0" layer="19" extent="1-1"/>
+<contactref element="CT5" pad="2"/>
+<contactref element="CT6" pad="2"/>
+<wire x1="22.27" y1="56" x2="22.27" y2="57.495" width="0.6096" layer="1"/>
+<wire x1="22.27" y1="57.495" x2="24.09" y2="59.315" width="0.6096" layer="1"/>
+<wire x1="19" y1="68.27" x2="22" y2="68.27" width="0.9144" layer="1"/>
+<wire x1="67.9" y1="54" x2="81" y2="48.73" width="0" layer="19" extent="1-1"/>
+<wire x1="60.85" y1="52" x2="67.9" y2="54" width="0" layer="19" extent="1-1"/>
 <wire x1="43.86" y1="43.84" x2="60.85" y2="52" width="0" layer="19" extent="1-1"/>
 <wire x1="32" y1="47.125" x2="43.86" y2="43.84" width="0" layer="19" extent="1-1"/>
-<wire x1="24.09" y1="59.315" x2="32" y2="47.125" width="0" layer="19" extent="1-1"/>
-<wire x1="21.875" y1="66" x2="24.09" y2="59.315" width="0" layer="19" extent="1-1"/>
-<wire x1="27.125" y1="62" x2="21.875" y2="66" width="0" layer="19" extent="1-1"/>
 <wire x1="22.27" y1="56" x2="32" y2="47.125" width="0" layer="19" extent="1-1"/>
-</signal>
-<signal name="N$1">
-<contactref element="CT5" pad="1"/>
-<contactref element="IC2" pad="5"/>
-<wire x1="18.89" y1="63.125" x2="20.125" y2="66" width="0" layer="19" extent="1-1"/>
+<wire x1="22" y1="68.27" x2="24.09" y2="59.315" width="0" layer="19" extent="1-1"/>
 </signal>
 <signal name="N$3">
 <contactref element="RT7" pad="3"/>
 <contactref element="RT72" pad="1"/>
-<wire x1="13.15" y1="58" x2="12.75" y2="60.5" width="0" layer="19" extent="1-1"/>
+<wire x1="12.75" y1="60.5" x2="12.75" y2="58.4" width="0.6096" layer="1"/>
+<wire x1="12.75" y1="58.4" x2="13.15" y2="58" width="0.6096" layer="1"/>
 </signal>
 <signal name="N$5">
@@
 <contactref element="RT73" pad="1"/>
 <contactref element="IC2" pad="7"/>
-<wire x1="14.85" y1="58" x2="15.15" y2="55" width="0" layer="19" extent="1-1"/>
-<wire x1="18.89" y1="60.585" x2="14.85" y2="58" width="0" layer="19" extent="1-1"/>
+<wire x1="14.85" y1="58" x2="15.15" y2="57.7" width="0.6096" layer="1"/>
+<wire x1="15.15" y1="57.7" x2="15.15" y2="55" width="0.6096" layer="1"/>
+<wire x1="18.89" y1="60.585" x2="16.585" y2="60.585" width="0.6096" layer="1"/>
+<wire x1="14.85" y1="58.85" x2="14.85" y2="58" width="0.6096" layer="1"/>
+<wire x1="16.585" y1="60.585" x2="14.85" y2="58.85" width="0.6096" layer="1"/>
 </signal>
 <signal name="N$6">
 <contactref element="IC2" pad="4"/>
 <contactref element="JP1" pad="1"/>
-<wire x1="24.09" y1="63.125" x2="6.73" y2="74" width="0" layer="19" extent="1-1"/>
+<wire x1="24.09" y1="63.125" x2="22.27" y2="76" width="0" layer="19" extent="1-1"/>
 </signal>
 <signal name="N$8">
 <contactref element="IC2" pad="2"/>
-<contactref element="CT6" pad="1"/>
 <contactref element="IC2" pad="6"/>
 <contactref element="RT7" pad="2"/>
 <contactref element="RT7" pad="1"/>
-<wire x1="24.09" y1="60.585" x2="28.875" y2="62" width="0" layer="19" extent="1-1"/>
-<wire x1="18.89" y1="61.855" x2="24.09" y2="60.585" width="0" layer="19" extent="1-1"/>
-<wire x1="15.25" y1="63" x2="18.89" y2="61.855" width="0" layer="19" extent="1-1"/>
-<wire x1="12.75" y1="65.5" x2="15.25" y2="63" width="0" layer="19" extent="1-1"/>
+<wire x1="15.25" y1="63" x2="16.395" y2="61.855" width="0.6096" layer="1"/>
+<wire x1="16.395" y1="61.855" x2="18.89" y2="61.855" width="0.6096" layer="1"/>
+<wire x1="12.75" y1="65.5" x2="15.25" y2="63" width="0.6096" layer="1"/>
+<contactref element="CT6" pad="1"/>
+<wire x1="18.89" y1="61.855" x2="20.855" y2="61.855" width="0.6096" layer="1"/>
+<wire x1="22" y1="63" x2="22" y2="65.73" width="0.6096" layer="1"/>
+<wire x1="20.855" y1="61.855" x2="22" y2="63" width="0.6096" layer="1"/>
+<wire x1="18.89" y1="61.855" x2="21.145" y2="61.855" width="0.6096" layer="1"/>
+<wire x1="22.415" y1="60.585" x2="24.09" y2="60.585" width="0.6096" layer="1"/>
+<wire x1="21.145" y1="61.855" x2="22.415" y2="60.585" width="0.6096" layer="1"/>
 </signal>
 <signal name="N$9">
@@
 <contactref element="IC2" pad="8"/>
 <contactref element="CPASST" pad="1"/>
-<wire x1="16.85" y1="55" x2="18.89" y2="59.315" width="0" layer="19" extent="1-1"/>
-<wire x1="19.73" y1="56" x2="16.85" y2="55" width="0" layer="19" extent="1-1"/>
+<wire x1="16.85" y1="55" x2="18.73" y2="55" width="0.9144" layer="1"/>
+<wire x1="18.73" y1="55" x2="19.73" y2="56" width="0.9144" layer="1"/>
+<wire x1="19.73" y1="56" x2="18" y2="57.73" width="0.6096" layer="1"/>
+<wire x1="18" y1="57.73" x2="18" y2="59.315" width="0.6096" layer="1"/>
+<wire x1="18.89" y1="59.315" x2="18" y2="59.315" width="0.6096" layer="1"/>
+</signal>
+<signal name="N$2">
+<contactref element="CT5" pad="1"/>
+<contactref element="IC2" pad="5"/>
+<wire x1="19" y1="65.73" x2="19" y2="63.235" width="0.6096" layer="1"/>
+<wire x1="19" y1="63.235" x2="18.89" y2="63.125" width="0.6096" layer="1"/>
 </signal>
 </signals>

Commit message: Add files via upload
Parts:
- added CPASST1, CPASST2, CPASST3, CT1, CT3, CT7: 0.1u, rcl:C025-024X044
- added CSENS1, CSENS2, CSENS3: (no value), rcl:C0603K
- added CT2, CT4, CT8: 1000p, rcl:C025-024X044
- added IC3, IC4, IC5: LM555D, linear:SO08
- added JP3, JP4, JP5, JP6, JP7, JP8: (no value), pinhead:1X02
- added RAMP3, RAMP5, RAMP7, RT2, RT5, RT9: 10k, rcl:R0603
- added RAMP4, RAMP6, RAMP8: 22k, rcl:R0603
- added RAMPD1, RAMPD2, RAMPD3, RAMPU1, RAMPU2, RAMPU3: 1, rcl:R0603
- added RT1, RT4, RT8: 10k, rcl:RTRIM74W
- added RT10, RT3, RT6: 1.5k, rcl:R0603
- added TNPN3, TNPN4, TNPN5, TNPN6, TNPN7, TNPN8, TPNP3, TPNP4, TPNP5, TPNP6, TPNP7, TPNP8: (no value), transistor:SOT23-BEC
- moved JP1 38.2 mm to (59.0, 72.0), turned to 270 degrees
- moved IC2 30.4 mm to (51.5, 66.2)
- moved CPASST 30.4 mm to (51.0, 61.0)
- moved CT5 30.4 mm to (49.0, 72.0)
- moved CT6 30.4 mm to (52.0, 72.0)
- moved RT7 30.4 mm to (44.0, 68.0)
- moved RT72 30.4 mm to (44.0, 63.0)
- moved RT73 30.4 mm to (46.0, 60.0)
- moved IC1 28.3 mm to (15.9, 43.6)
- moved CPASS 28.0 mm to (4.00, 47.0)
- moved CSENS 12.2 mm to (79.0, 64.0)
- moved JP2 12.2 mm to (83.0, 62.0)
- moved RAMP1 12.2 mm to (62.0, 64.0)
- moved RAMP2 12.2 mm to (62.0, 67.0)
- moved RAMPD 12.2 mm to (75.0, 66.0)
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Connections:
- removed net +5V/1: CPASST.1, IC2.8, RT73.2
- new net +5V: CPASST.1, CPASST1.1, CPASST2.1, CPASST3.1, IC2.8, IC3.8, IC4.8, IC5.8, RT10.2, RT3.2, RT6.2, RT73.2
- new net N$1: RT1.3, RT2.1
- new net N$11: IC3.4, JP3.1
- new net N$12: CT2.1, IC3.2, IC3.6, RT1.1, RT1.2
- new net N$15: RAMP3.2, RAMP4.1
- new net N$17: RAMPU1.2, TNPN3.E, TNPN4.B
- new net N$18: TNPN3.B, TNPN4.C, TPNP3.C, TPNP4.B
- new net N$19: RAMPD1.1, TPNP3.B, TPNP4.E
- new net N$20: CSENS1.1, RAMP4.2, RAMPD1.2, RAMPU1.1, TNPN4.E, TPNP3.E
- new net N$21: CSENS1.2, JP4.1
- new net N$22: CT1.1, IC3.5
- new net N$23: RT4.3, RT5.1
- new net N$24: IC4.7, RT5.2, RT6.1
- new net N$25: IC4.4, JP5.1
- new net N$26: CT4.1, IC4.2, IC4.6, RT4.1, RT4.2
- new net N$27: RAMP5.2, RAMP6.1
- new net N$28: RAMPU2.2, TNPN5.E, TNPN6.B
- new net N$29: TNPN5.B, TNPN6.C, TPNP5.C, TPNP6.B
- new net N$30: RAMPD2.1, TPNP5.B, TPNP6.E
- new net N$31: CSENS2.1, RAMP6.2, RAMPD2.2, RAMPU2.1, TNPN6.E, TPNP5.E
- new net N$32: CSENS2.2, JP6.1
- new net N$33: CT3.1, IC4.5
- new net N$34: RT8.3, RT9.1
- new net N$35: IC5.7, RT10.1, RT9.2
- new net N$36: IC5.4, JP7.1
- new net N$37: CT8.1, IC5.2, IC5.6, RT8.1, RT8.2
- new net N$38: RAMP7.2, RAMP8.1
- new net N$39: RAMPU3.2, TNPN7.E, TNPN8.B
- new net N$40: TNPN7.B, TNPN8.C, TPNP7.C, TPNP8.B
- new net N$41: RAMPD3.1, TPNP7.B, TPNP8.E
- new net N$42: CSENS3.1, RAMP8.2, RAMPD3.2, RAMPU3.1, TNPN8.E, TPNP7.E
- new net N$43: CSENS3.2, JP8.1
- new net N$44: CT7.1, IC5.5
- net +9V: now also TNPN3.C, TNPN5.C, TNPN7.C
- net DGND: now also CPASST1.2, CPASST2.2, CPASST3.2, CT1.2, CT2.2, CT3.2, CT4.2, CT7.2, CT8.2, IC3.1, IC4.1, IC5.1, JP4.2, JP6.2, JP8.2, RAMP3.1, RAMP5.1, RAMP7.1, TPNP4.C, TPNP6.C, TPNP8.C
- net N$4: no longer IC1.2
- net N$7: no longer IC1.1
- net N$9: now also IC3.7, RT2.2, RT3.1; no longer IC1.3, IC2.3
Routing:
- net +5V: track 0.00 -> 32.9 mm
- net N$42: track 0.00 -> 23.5 mm
- net N$31: track 0.00 -> 23.5 mm
- net N$20: track 0.00 -> 23.5 mm
- net DGND: track 7.07 -> 28.3 mm
- net N$12: track 0.00 -> 19.7 mm
- net N$37: track 0.00 -> 19.7 mm
- net N$26: track 0.00 -> 19.7 mm
- net N$29: track 0.00 -> 13.2 mm
- net N$40: track 0.00 -> 13.2 mm
- net N$18: track 0.00 -> 13.2 mm
- net N$39: track 0.00 -> 11.2 mm, vias 0 -> 2
- net N$28: track 0.00 -> 11.2 mm, vias 0 -> 2
- net N$17: track 0.00 -> 11.2 mm, vias 0 -> 2
- net N$9: track 0.00 -> 8.73 mm
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
Commit message: Add files via upload
Parts:
- removed JP1, JP3, JP5, JP7: (no value), pinhead:1X02
- added JP9: (no value), pinhead:1X04
- moved CPASS 33.5 mm to (37.0, 41.0)
- moved IC1 32.0 mm to (47.9, 42.6)
- moved CPASST3 26.8 mm to (39.0, 28.0), turned to 90 degrees
- moved CPASST 26.7 mm to (25.0, 55.0), turned to 270 degrees
- moved IC5 25.5 mm to (34.8, 28.5), turned to 180 degrees
- moved CT8 25.5 mm to (29.0, 26.0), turned to 270 degrees
- moved IC2 24.3 mm to (30.2, 54.5), turned to 0 degrees
- moved CT6 24.0 mm to (35.0, 55.0)
- moved RAMP7 24.0 mm to (61.0, 31.0), turned to 0 degrees
- moved RT3 23.1 mm to (40.0, 64.0), turned to 180 degrees
- moved RT2 22.6 mm to (40.0, 67.0)
- moved RT10 21.8 mm to (40.0, 24.0)
- moved RT73 21.0 mm to (25.0, 60.0), turned to 180 degrees
- moved CPASST1 20.8 mm to (40.0, 60.0), turned to 270 degrees
- moved CT7 20.6 mm to (29.0, 20.0), turned to 270 degrees
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Connections:
- new net N$45: IC1.5, IC2.3
- new net N$46: IC1.3, IC3.3
- new net N$47: IC1.12, IC4.3
- new net N$48: IC1.9, IC5.3
- net N$11: now also IC4.4, JP9.3; no longer IC3.4, JP3.1
- net N$15: now also IC1.2
- net N$18: now also IC1.1
- net N$25: now also IC3.4, JP9.2; no longer IC4.4, JP5.1
- net N$27: now also IC1.13
- net N$29: now also IC1.14
- net N$36: now also IC2.4, JP9.1; no longer IC5.4, JP7.1
- net N$38: now also IC1.10
- net N$4: now also IC1.6
- net N$40: now also IC1.8
- net N$6: now also IC5.4, JP9.4; no longer IC2.4, JP1.1
- net N$7: now also IC1.7
Routing:
- net N$7: track 13.2 -> 46.0 mm
- net N$40: track 13.2 -> 45.9 mm
- net N$25: track 0.00 -> 28.6 mm
- net N$4: track 3.00 -> 30.3 mm, vias 0 -> 1
- net N$11: track 0.00 -> 24.0 mm
- net N$45: track 0.00 -> 21.1 mm, vias 0 -> 1
- net N$38: track 3.00 -> 23.2 mm
- net +9V: track 3.31 -> 17.6 mm
- net N$48: track 0.00 -> 13.7 mm, vias 0 -> 1
- net N$46: track 0.00 -> 13.0 mm, vias 0 -> 1
- net DGND: track 28.3 -> 15.3 mm
- net N$18: track 13.2 -> 24.7 mm
- net N$29: track 13.2 -> 24.5 mm
- net N$36: track 0.00 -> 11.2 mm
- net N$15: track 3.00 -> 14.2 mm
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
Commit message: Add files via upload
Parts:
- added C1, C2, C3, C4: (no value), rcl:C025-024X044
- added JP3: (no value), pinhead:2X02
- added L1, L2: (no value), rcl:0207/7
- moved CPASS 21.2 mm to (58.0, 44.0), turned to 90 degrees
- moved RAMP5 5.70 mm to (65.5, 42.5), turned to 180 degrees
- moved JP9 4.47 mm to (31.0, 41.0)
- moved RT5 2.24 mm to (54.0, 19.0), turned to 90 degrees
- moved RT9 2.24 mm to (38.0, 20.0), turned to 90 degrees
- moved RAMP7 2.00 mm to (63.0, 31.0), turned to 180 degrees
- moved CPASST2 1.00 mm to (54.0, 27.0)
- moved CPASST3 1.00 mm to (38.0, 28.0)
- moved CT3 1.00 mm to (44.0, 20.0)
- moved CT4 1.00 mm to (44.0, 25.0)
- moved CT7 1.00 mm to (28.0, 20.0)
- moved CT8 1.00 mm to (28.0, 26.0)
- moved IC4 1.00 mm to (48.8, 27.5)
- moved IC5 1.00 mm to (33.8, 28.5)
- moved RT10 1.00 mm to (39.0, 24.0)
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Connections:
- new net N$49: C2.1, JP3.3, L1.1
- new net N$51: C1.1, JP3.4, L2.1
- net +5V: now also C4.1, L1.2
- net +9V: now also C3.1, L2.2
- net DGND: now also C1.2, C2.2, C3.2, C4.2, JP3.1, JP3.2
Routing:
- net +9V: track 17.6 -> 98.1 mm, vias 0 -> 5
- net DGND: track 15.3 -> 31.0 mm, vias 0 -> 9
- net N$51: track 0.00 -> 9.13 mm
- net N$49: track 0.00 -> 8.58 mm
- net N$11: track 24.0 -> 19.9 mm
- net N$23: track 6.60 -> 2.82 mm
- net N$36: track 11.2 -> 7.57 mm
- net N$3: track 6.16 -> 2.71 mm
- net +5V: track 29.3 -> 25.9 mm
- net N$25: track 28.6 -> 25.4 mm
- net N$34: track 5.87 -> 2.67 mm
- net N$1: track 5.16 -> 2.77 mm
- net N$27: track 13.9 -> 15.7 mm
- net N$6: track 8.18 -> 6.46 mm
- net N$26: track 20.4 -> 19.5 mm
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- added copper zone on layer 1, net +5V
- added copper zone on layer 1, net +9V
- added copper zone on layer 16, net DGND
Other:
- board size 100 x 80 mm -> 70 x 66 mm
