File: Eagle/PhasedArrayTransmittor/PhasedArrayTransmittor.sch (EAGLE design)
At the start: 18 parts, among them IC1 OP400P, IC2 LM555D

Commit message: Add files via upload
Parts:
- added CPASS: 0.1u, rcl:C-EUC0603K
- added CPASST: 0.1u, rcl:C-EU025-024X044
- renumbered C1 to CT5, C2 to CT6, C3 to CSENS, R1 to RT7, R2 to RT72, R3 to RT73, R4 to RAMP1, R5 to RAMP2, R6 to RAMPU, R7 to RAMPD, T1 to TNPN2, T2 to TNPN1, T3 to TPNP1, T4 to TPNP2
Connections:
- net +5V/1: now also CPASST.1
- net +9V: now also CPASS.1
- net DGND: now also CPASS.2, CPASST.2

Commit message: Add files via upload
Parts:
- CT5, CT6: device rcl:C-EUC0603K -> rcl:C-EU025-024X044

Commit message: Add files via upload
Parts:
- added CPASST1, CPASST2, CPASST3, CT1, CT3, CT7: 0.1u, rcl:C-EU025-024X044
- added CSENS1, CSENS2, CSENS3: (no value), rcl:C-EUC0603K
- added CT2, CT4, CT8: 1000p, rcl:C-EU025-024X044
- added IC3, IC4, IC5: LM555D, linear:LM555D
- added JP3, JP4, JP5, JP6, JP7, JP8: (no value), pinhead:PINHD-1X2
- added RAMP3, RAMP5, RAMP7, RT2, RT5, RT9: 10k, rcl:R-EU_R0603
- added RAMP4, RAMP6, RAMP8: 22k, rcl:R-EU_R0603
- added RAMPD1, RAMPD2, RAMPD3, RAMPU1, RAMPU2, RAMPU3: 1, rcl:R-EU_R0603
- added RT1, RT4, RT8: 10k, rcl:R-TRIMM74W
- added RT10, RT3, RT6: 1.5k, rcl:R-EU_R0603
- added TNPN3, TNPN4, TNPN5, TNPN6, TNPN7, TNPN8: (no value), transistor:BC817-16-NPN-SOT23-BEC
- added TPNP3, TPNP4, TPNP5, TPNP6, TPNP7, TPNP8: (no value), transistor:BC807-16-PNP-SOT23-BEC
Connections:
- removed net +5V/1: CPASST.1, IC2.V+, RT73.2
- new net +5V: CPASST.1, CPASST1.1, CPASST2.1, CPASST3.1, IC2.V+, IC3.V+, IC4.V+, IC5.V+, RT10.2, RT3.2, RT6.2, RT73.2
- new net N$1: RT1.E, RT2.1
- new net N$11: IC3.R, JP3.1
- new net N$12: CT2.1, IC3.THR, IC3.TR, RT1.A, RT1.S
- new net N$15: RAMP3.2, RAMP4.1
- new net N$17: RAMPU1.2, TNPN3.E, TNPN4.B
- new net N$18: TNPN3.B, TNPN4.C, TPNP3.C, TPNP4.B
- new net N$19: RAMPD1.1, TPNP3.B, TPNP4.E
- new net N$20: CSENS1.1, RAMP4.2, RAMPD1.2, RAMPU1.1, TNPN4.E, TPNP3.E
- new net N$21: CSENS1.2, JP4.1
- new net N$22: CT1.1, IC3.CV
- new net N$23: RT4.E, RT5.1
- new net N$24: IC4.DIS, RT5.2, RT6.1
- new net N$25: IC4.R, JP5.1
- new net N$26: CT4.1, IC4.THR, IC4.TR, RT4.A, RT4.S
- new net N$27: RAMP5.2, RAMP6.1
- new net N$28: RAMPU2.2, TNPN5.E, TNPN6.B
- new net N$29: TNPN5.B, TNPN6.C, TPNP5.C, TPNP6.B
- new net N$30: RAMPD2.1, TPNP5.B, TPNP6.E
- new net N$31: CSENS2.1, RAMP6.2, RAMPD2.2, RAMPU2.1, TNPN6.E, TPNP5.E
- new net N$32: CSENS2.2, JP6.1
- new net N$33: CT3.1, IC4.CV
- new net N$34: RT8.E, RT9.1
- new net N$35: IC5.DIS, RT10.1, RT9.2
- new net N$36: IC5.R, JP7.1
- new net N$37: CT8.1, IC5.THR, IC5.TR, RT8.A, RT8.S
- new net N$38: RAMP7.2, RAMP8.1
- new net N$39: RAMPU3.2, TNPN7.E, TNPN8.B
- new net N$40: TNPN7.B, TNPN8.C, TPNP7.C, TPNP8.B
- new net N$41: RAMPD3.1, TPNP7.B, TPNP8.E
- new net N$42: CSENS3.1, RAMP8.2, RAMPD3.2, RAMPU3.1, TNPN8.E, TPNP7.E
- new net N$43: CSENS3.2, JP8.1
- new net N$44: CT7.1, IC5.CV
- net +9V: now also TNPN3.C, TNPN5.C, TNPN7.C
- net DGND: now also CPASST1.2, CPASST2.2, CPASST3.2, CT1.2, CT2.2, CT3.2, CT4.2, CT7.2, CT8.2, IC3.GND, IC4.GND, IC5.GND, JP4.2, JP6.2, JP8.2, RAMP3.1, RAMP5.1, RAMP7.1, TPNP4.C, TPNP6.C, TPNP8.C
- net N$4: no longer IC1A.-IN
- net N$7: no longer IC1A.OUT
- net N$9: now also IC3.DIS, RT2.2, RT3.1; no longer IC1A.+IN, IC2.Q
Other:
- moved on the sheet: CPASS, IC1A

Commit message: Add files via upload
Parts:
- removed JP1, JP3, JP5, JP7: (no value), pinhead:PINHD-1X2
- added JP9: (no value), pinhead:PINHD-1X4
Connections:
- new net N$45: IC1B.+IN, IC2.Q
- new net N$46: IC1A.+IN, IC3.Q
- new net N$47: IC1D.+IN, IC4.Q
- new net N$48: IC1C.-IN, IC5.Q
- net N$11: now also IC4.R, JP9.3; no longer IC3.R, JP3.1
- net N$15: now also IC1A.-IN
- net N$18: now also IC1A.OUT
- net N$25: now also IC3.R, JP9.2; no longer IC4.R, JP5.1
- net N$27: now also IC1D.-IN
- net N$29: now also IC1D.OUT
- net N$36: now also IC2.R, JP9.1; no longer IC5.R, JP7.1
- net N$38: now also IC1C.+IN
- net N$4: now also IC1B.-IN
- net N$40: now also IC1C.OUT
- net N$6: now also IC5.R, JP9.4; no longer IC2.R, JP1.1
- net N$7: now also IC1B.OUT
Other:
- moved on the sheet: IC1A

Commit message: Add files via upload
Parts:
- added C1, C2, C3, C4: (no value), rcl:C-EU025-024X044
- added JP3: (no value), pinhead:PINHD-2X2
- added L1, L2: (no value), rcl:L-EU0207/7
Connections:
- new net N$49: C2.1, JP3.3, L1.1
- new net N$51: C1.1, JP3.4, L2.1
- net +5V: now also C4.1, L1.2
- net +9V: now also C3.1, L2.2
- net DGND: now also C1.2, C2.2, C3.2, C4.2, JP3.1, JP3.2
Other:
- moved on the sheet: CPASS
