File: Eagle/PhasedArray2/UltrasonicSensor/UltrasonicSensor.brd (EAGLE design)
At the start: 100 x 80 mm, 55 parts, among them IC3 OP400P

Commit message: Add files via upload
Parts:
- removed C1PASS2: 0.1u, rcl:C025-024X044
- removed C1SENSOR2, C2AMP3: 0.1u, rcl:C0603K
- removed C3F3, C4F3, C5F3, C6F3: 1000p, rcl:C0603K
- removed C7: 0.1u, rcl:C1608
- removed IC3: OP400P, linear:DIL14
- removed JP3: (no value), pinhead:1X02
- removed R11F3: 15k, rcl:R0603
- removed R12F3, R13F3: 330, rcl:R0603
- removed R14F3: 39k, rcl:0207/7
- removed R15F3: 47k, rcl:0207/7
- removed R1AMP3, R3AMP1M2, R6AMP2M2, R7AMP3, R8AMP3: 10k, rcl:R0603
- removed R1F3: 15k, rcl:0207/7
- removed R2: 500k, rcl:PT-10
- removed R2AMP3: 1M, rcl:R0603
- added C14: 0.1u, rcl:C1608
- added VR1: 3361P-1-504GLF, 3361P-1-504GLF:3361P1253GLF
- C6: value 10u -> 0.1u; device rcl:C2012 -> rcl:C1608
- JP1: device pinhead:1X02 -> pinhead:1X01
- R8: value 15k -> 18k
- R9: value 330 -> 390
- moved R10 190.0 mm to (73.8, 66.6)
- moved R12 189.1 mm to (65.0, 59.4), turned to 90 degrees
- moved C10 189.1 mm to (76.7, 67.1), turned to 270 degrees
- moved C13 187.5 mm to (68.0, 64.2), turned to 180 degrees
- moved R11 187.5 mm to (67.7, 59.4), turned to 270 degrees
- moved R8 186.8 mm to (79.0, 67.1), turned to 90 degrees
- moved R7 184.1 mm to (81.5, 67.1), turned to 270 degrees
- moved R9 182.5 mm to (68.0, 67.1), turned to 180 degrees
- moved C11 179.7 mm to (71.0, 67.0), turned to 270 degrees
- moved R6 174.1 mm to (91.0, 63.7), turned to 270 degrees
- moved IC1 171.1 mm to (79.0, 61.0)
- moved R5 169.2 mm to (88.3, 63.7), turned to 270 degrees
- moved C6 144.3 mm to (89.2, 55.3), turned to 270 degrees
- moved C9 136.7 mm to (85.0, 67.5), turned to 180 degrees
- moved R3 134.3 mm to (86.1, 59.6), turned to 270 degrees
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Connections:
- removed net N$1: IC3.7, R1F3.1, R2AMP3.2
- removed net N$32: R2.2, R2.3, R8AMP3.2
- removed net N$33: IC3.6, R1AMP3.2, R2AMP3.1
- removed net N$35: IC3.2, R7AMP3.2, R8AMP3.1
- removed net N$36: IC3.3, R6AMP2M2.2
- removed net N$37: C1SENSOR2.2, R1AMP3.1
- removed net N$38: C2AMP3.2, R7AMP3.1
- removed net N$40: C2AMP3.1, C3F3.2, IC3.14, R15F3.2
- removed net N$41: C5F3.2, IC3.9, R14F3.1
- removed net N$42: C4F3.2, IC3.13, R15F3.1
- removed net N$43: C3F3.1, C4F3.1, R11F3.2, R13F3.2
- removed net N$44: C6F3.2, IC3.8, R11F3.1, R14F3.2
- removed net N$45: C5F3.1, C6F3.1, R12F3.2, R1F3.2
- removed net N$46: IC3.5, R3AMP1M2.2
- removed net N$47: C1SENSOR2.1, JP1.1
- removed net N$48: IC3.1, R2.1
- removed net VMM: IC3.10, IC3.12, JP1.2, R3AMP1M2.1, R6AMP2M2.1
- new net N$16: IC1.1, JP1.1, VR1.2, VR1.3
- net +9V: no longer C6.2, C7.2, JP3.2
- net AGND: now also C14.2, C6.2; no longer C1PASS2.2, IC3.11, R12F3.1, R13F3.1
- net GND: no longer C6.1, C7.1, JP3.1
- net N$15: now also VR1.1
- net VCC: no longer C1PASS2.1, IC3.4
- net VCC/2: now also C14.1, C6.1
Routing:
- net VCC/2: track 0.00 -> 111.1 mm, vias 0 -> 2
- net VCC: track 0.00 -> 39.3 mm, vias 0 -> 2
- net N$16: track 0.00 -> 32.8 mm
- net AGND: track 0.00 -> 20.5 mm, vias 0 -> 6
- net N$15: track 0.00 -> 13.9 mm
- net N$9: track 0.00 -> 13.7 mm
- net N$12: track 0.00 -> 11.2 mm
- net N$5: track 0.00 -> 11.2 mm
- net N$11: track 0.00 -> 9.42 mm
- net N$14: track 0.00 -> 9.36 mm
- net N$8: track 0.00 -> 9.32 mm
- net N$7: track 0.00 -> 8.20 mm
- net N$10: track 0.00 -> 8.00 mm
- net N$13: track 0.00 -> 4.69 mm
- net N$2: track 0.00 -> 4.18 mm
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- added copper zone on layer 16, net AGND

Commit message: Add files via upload
Parts:
- added C16, C24, C25, C26, C27, C28, C33, C34, C35, C36, C37, C42, C43, C44, C7: 0.1u, rcl:C1608
- added C18, C21, C22, C23, C29, C30, C31, C32, C38, C39, C40, C41: 1000p, rcl:C1608
- added IC2, IC3, IC4: (no value), linear3:NJM2734M
- added JP3, JP6, JP8: (no value), pinhead:1X02
- added JP4, JP7, JP9: (no value), pinhead:1X01
- added R13, R23, R33: 15k, rcl:R0603
- added R14, R24, R34: 330, rcl:R0603
- added R15, R25, R35: 39k, rcl:R0603
- added R16, R26, R36: 18k, rcl:R0603
- added R17, R27, R37: 390, rcl:R0603
- added R18, R28, R38: 47k, rcl:R0603
- added R19, R2, R20, R21, R29, R30, R31, R39, R40: 10k, rcl:R0603
- added R22, R32, R4: 1M, rcl:R0603
- added VR2, VR3, VR4: 3361P-1-504GLF, 3361P-1-504GLF:3361P1253GLF
- moved R11 8.06 mm to (66.7, 67.4)
- moved R12 8.06 mm to (64.0, 67.4)
- moved C1 8.06 mm to (70.6, 69.1)
- moved C10 8.06 mm to (75.7, 75.1)
- moved C11 8.06 mm to (70.0, 75.0)
- moved C13 8.06 mm to (67.0, 72.2)
- moved C14 8.06 mm to (71.9, 63.1)
- moved C2 8.06 mm to (91.9, 67.6)
- moved C6 8.06 mm to (88.2, 63.3)
- moved C9 8.06 mm to (84.0, 75.5)
- moved IC1 8.06 mm to (78.0, 69.0)
- moved JP1 8.06 mm to (48.0, 71.0)
- moved R1 8.06 mm to (88.5, 67.1)
- moved R10 8.06 mm to (72.8, 74.6)
- moved R3 8.06 mm to (85.1, 67.6)
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Connections:
- new net N$1: C16.2, R2.1
- new net N$17: C16.1, JP3.2
- new net N$18: IC2.7, R13.2, R4.1
- new net N$19: C18.1, C21.1, R13.1, R14.1
- new net N$20: IC2.6, R2.2, R4.2
- new net N$21: C18.2, IC2.9, R15.2
- new net N$22: C21.2, IC2.8, R15.1, R16.2
- new net N$23: C22.1, C23.1, R16.1, R17.1
- new net N$24: C22.2, IC2.13, R18.2
- new net N$25: C23.2, C24.1, IC2.14, R18.1
- new net N$26: C24.2, R19.1
- new net N$27: IC2.2, R19.2, R20.1
- new net N$28: R20.2, VR2.1
- new net N$29: IC2.1, JP4.1, VR2.2, VR2.3
- new net N$30: C28.2, R21.1
- new net N$31: C28.1, JP6.2
- new net N$32: IC3.7, R22.1, R23.2
- new net N$33: C29.1, C30.1, R23.1, R24.1
- new net N$35: IC3.6, R21.2, R22.2
- new net N$36: C29.2, IC3.9, R25.2
- new net N$37: C30.2, IC3.8, R25.1, R26.2
- new net N$38: C31.1, C32.1, R26.1, R27.1
- new net N$39: C31.2, IC3.13, R28.2
- new net N$40: C32.2, C33.1, IC3.14, R28.1
- new net N$41: C33.2, R29.1
- new net N$42: IC3.2, R29.2, R30.1
- new net N$43: R30.2, VR3.1
- new net N$44: IC3.1, JP7.1, VR3.2, VR3.3
- new net N$45: C37.2, R31.1
- new net N$46: C37.1, JP8.2
- new net N$47: IC4.7, R32.1, R33.2
- new net N$48: C38.1, C39.1, R33.1, R34.1
- new net N$49: IC4.6, R31.2, R32.2
- new net N$50: C38.2, IC4.9, R35.2
- new net N$51: C39.2, IC4.8, R35.1, R36.2
- new net N$52: C40.1, C41.1, R36.1, R37.1
- new net N$53: C40.2, IC4.13, R38.2
- new net N$54: C41.2, C42.1, IC4.14, R38.1
- new net N$55: C42.2, R39.1
- new net N$56: IC4.2, R39.2, R40.1
- new net N$57: R40.2, VR4.1
- new net N$58: IC4.1, JP9.1, VR4.2, VR4.3
- net AGND: now also C25.2, C26.2, C27.1, C34.2, C35.2, C36.1, C43.2, C44.2, C7.1, IC2.11, IC3.11, IC4.11, R14.2, R17.2, R24.2, R27.2, R34.2, R37.2
- net VCC: now also C27.2, C36.2, C7.2, IC2.4, IC3.4, IC4.4
- net VCC/2: now also C25.1, C26.1, C34.1, C35.1, C43.1, C44.1, IC2.10, IC2.12, IC2.3, IC2.5, IC3.10, IC3.12, IC3.3, IC3.5, IC4.10, IC4.12, IC4.3, IC4.5, JP3.1, JP6.1, JP8.1
Routing:
- net VCC/2: track 111.1 -> 444.3 mm, vias 2 -> 8
- net VCC: track 39.3 -> 157.1 mm, vias 2 -> 8
- net AGND: track 20.5 -> 82.0 mm, vias 6 -> 24
- net N$29: track 0.00 -> 32.8 mm
- net N$58: track 0.00 -> 32.8 mm
- net N$44: track 0.00 -> 32.8 mm
- net N$57: track 0.00 -> 13.9 mm
- net N$43: track 0.00 -> 13.9 mm
- net N$28: track 0.00 -> 13.9 mm
- net N$56: track 0.00 -> 13.7 mm
- net N$27: track 0.00 -> 13.7 mm
- net N$42: track 0.00 -> 13.7 mm
- net N$38: track 0.00 -> 11.2 mm
- net N$23: track 0.00 -> 11.2 mm
- net N$52: track 0.00 -> 11.2 mm
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
Commit message: Add files via upload
Parts:
- removed JP4, JP7, JP9: (no value), pinhead:1X01
- added C45, C46: 10u, rcl:C2012
- added C47: 1000p, rcl:C1608
- added PS3: ADP7112ACBZ-5.0-R7, ADP7112ACBZ-3.3-R7:BGA6C40P2X3_95X116X56
- JP1: device pinhead:1X01 -> pinhead:1X08
- moved JP1 46.8 mm to (17.0, 36.0), turned to 270 degrees
- moved JP5 30.9 mm to (2.60, 44.8), turned to 90 degrees
- moved C19 26.9 mm to (5.98, 44.4), turned to 90 degrees
- moved C14 25.5 mm to (46.9, 58.1)
- moved C8 25.5 mm to (59.7, 66.7)
- moved C1 25.5 mm to (45.6, 64.1)
- moved C10 25.5 mm to (50.7, 70.1)
- moved C11 25.5 mm to (45.0, 70.0)
- moved C13 25.5 mm to (42.0, 67.2)
- moved C2 25.5 mm to (66.9, 62.6)
- moved C6 25.5 mm to (63.2, 58.3)
- moved IC1 25.5 mm to (53.0, 64.0)
- moved R1 25.5 mm to (63.5, 62.1)
- moved R10 25.5 mm to (47.8, 69.6)
- moved R11 25.5 mm to (41.7, 62.4)
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Connections:
- new net N$59: C47.1, PS3.B1
- net +9V: now also C45.1, PS3.A1, PS3.C1
- net AGND: now also C46.2
- net GND: now also C45.2, C47.2, PS3.C2
- net N$16: now also JP1.2; no longer JP1.1
- net N$29: now also JP1.4; no longer JP4.1
- net N$44: now also JP1.6; no longer JP7.1
- net N$58: now also JP1.8; no longer JP9.1
- net VCC: now also C46.1, PS3.A2, PS3.B2
- net VCC/2: now also JP1.1, JP1.3, JP1.5, JP1.7
Routing:
- net +9V: track 0.00 -> 119.3 mm
- net VCC: track 157.1 -> 263.6 mm, vias 8 -> 12
- net VCC/2: track 444.3 -> 550.4 mm, vias 8 -> 15
- net AGND: track 82.0 -> 112.5 mm, vias 24 -> 27
- net GND: track 0.00 -> 29.2 mm, vias 0 -> 7
- net N$16: track 32.8 -> 52.4 mm, vias 0 -> 2
- net N$58: track 32.8 -> 49.8 mm, vias 0 -> 2
- net N$29: track 32.8 -> 41.5 mm, vias 0 -> 1
- net N$44: track 32.8 -> 39.7 mm
- net N$59: track 0.00 -> 3.69 mm
- net N$34: track 0.00 -> 3.54 mm
- net N$6: track 0.00 -> 3.36 mm
- added copper zone on layer 16, net GND
Other:
- board size 100 x 80 mm -> 80 x 73 mm

Commit message: Add files via upload
Routing:
- net AGND: track 112.5 -> 111.7 mm
Changed lines of the file:
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@@
 </class>
 </classes>
-<designrules name="default">
+<designrules name="Elecrow_2-layer_PCB_eagle_rule">
 <description language="de">&lt;b&gt;EAGLE Design Rules&lt;/b&gt;
 &lt;p&gt;
@@
 necessary adjustments and save your customized
 design rules under a new name.</description>
+<description language="zh">&lt;b&gt;Elecrow PCB EAGLE Design Rules&lt;/b&gt;
+</description>
 <param name="layerSetup" value="(1*16)"/>
 <param name="mtCopper" value="0.035mm 0.035mm 0.035mm 0.035mm 0.035mm 0.035mm 0.035mm 0.035mm 0.035mm 0.035mm 0.035mm 0.035mm 0.035mm 0.035mm 0.035mm 0.035mm"/>
-<param name="mtIsolate" value="1.5mm 0.15mm 0.2mm 0.15mm 0.2mm 0.15mm 0.2mm 0.15mm 0.2mm 0.15mm 0.2mm 0.15mm 0.2mm 0.15mm 0.2mm"/>
+<param name="mtIsolate" value="1.6mm 1.2mm 0.2mm 0.15mm 0.2mm 0.15mm 0.2mm 0.15mm 0.2mm 0.15mm 0.2mm 0.15mm 0.2mm 0.15mm 0.2mm"/>
 <param name="mdWireWire" value="6mil"/>
 <param name="mdWirePad" value="6mil"/>
@@
 <param name="mdPadPad" value="6mil"/>
 <param name="mdPadVia" value="6mil"/>
-<param name="mdViaVia" value="6mil"/>
-<param name="mdSmdPad" value="6mil"/>
-<param name="mdSmdVia" value="6mil"/>
-<param name="mdSmdSmd" value="6mil"/>
-<param name="mdViaViaSameLayer" value="6mil"/>
+<param name="mdViaVia" value="8mil"/>
+<param name="mdSmdPad" value="0mil"/>
+<param name="mdSmdVia" value="0mil"/>
+<param name="mdSmdSmd" value="0mil"/>
+<param name="mdViaViaSameLayer" value="8mil"/>
 <param name="mnLayersViaInSmd" value="2"/>
-<param name="mdCopperDimension" value="40mil"/>
-<param name="mdDrill" value="6mil"/>
+<param name="mdCopperDimension" value="20mil"/>
+<param name="mdDrill" value="10mil"/>
 <param name="mdSmdStop" value="0mil"/>
 <param name="msWidth" value="6mil"/>
-<param name="msDrill" value="0.35mm"/>
-<param name="msMicroVia" value="9.99mm"/>
+<param name="msDrill" value="12mil"/>
+<param name="msMicroVia" value="12mil"/>
 <param name="msBlindViaRatio" value="0.5"/>
 <param name="rvPadTop" value="0.25"/>
@@
 <param name="rvMicroViaOuter" value="0.25"/>
 <param name="rvMicroViaInner" value="0.25"/>
-<param name="rlMinPadTop" value="10mil"/>
+<param name="rlMinPadTop" value="6mil"/>
 <param name="rlMaxPadTop" value="20mil"/>
-<param name="rlMinPadInner" value="10mil"/>
+<param name="rlMinPadInner" value="6mil"/>
 <param name="rlMaxPadInner" value="20mil"/>
-<param name="rlMinPadBottom" value="10mil"/>
+<param name="rlMinPadBottom" value="6mil"/>
 <param name="rlMaxPadBottom" value="20mil"/>
-<param name="rlMinViaOuter" value="8mil"/>
+<param name="rlMinViaOuter" value="6mil"/>
 <param name="rlMaxViaOuter" value="20mil"/>
-<param name="rlMinViaInner" value="8mil"/>
+<param name="rlMinViaInner" value="6mil"/>
 <param name="rlMaxViaInner" value="20mil"/>
 <param name="rlMinMicroViaOuter" value="4mil"/>
@@
 <param name="psTop" value="-1"/>
 <param name="psBottom" value="-1"/>
-<param name="psFirst" value="-1"/>
+<param name="psFirst" value="0"/>
 <param name="psElongationLong" value="100"/>
 <param name="psElongationOffset" value="100"/>
 <param name="mvStopFrame" value="1"/>
 <param name="mvCreamFrame" value="0"/>
-<param name="mlMinStopFrame" value="4mil"/>
-<param name="mlMaxStopFrame" value="4mil"/>
+<param name="mlMinStopFrame" value="0mil"/>
+<param name="mlMaxStopFrame" value="0mil"/>
 <param name="mlMinCreamFrame" value="0mil"/>
 <param name="mlMaxCreamFrame" value="0mil"/>
-<param name="mlViaStopLimit" value="0mil"/>
+<param name="mlViaStopLimit" value="100mil"/>
 <param name="srRoundness" value="0"/>
 <param name="srMinRoundness" value="0mil"/>
@@
 <param name="checkAngle" value="0"/>
 <param name="checkFont" value="1"/>
-<param name="checkRestrict" value="1"/>
+<param name="checkRestrict" value="0"/>
 <param name="checkStop" value="0"/>
 <param name="checkValues" value="0"/>
@@
 <wire x1="18.5" y1="54.3" x2="19.7" y2="54.3" width="0.254" layer="16"/>
 <wire x1="19.7" y1="54.3" x2="20" y2="54" width="0.254" layer="16"/>
-<wire x1="45.3" y1="57.2" x2="45.8" y2="57.2" width="0.254" layer="16"/>
-<wire x1="45.8" y1="57.2" x2="46" y2="57" width="0.254" layer="16"/>
-<wire x1="46.9" y1="57.25" x2="46.85" y2="57.2" width="0.6096" layer="1"/>
-<wire x1="46.85" y1="57.2" x2="45.3" y2="57.2" width="0.6096" layer="1"/>
 <wire x1="21" y1="13" x2="21" y2="19" width="0.254" layer="16"/>
+<wire x1="46.9" y1="57.25" x2="46.779290625" y2="57.2" width="0.508" layer="1" curve="-45"/>
+<wire x1="46.779290625" y1="57.2" x2="45.3" y2="57.2" width="0.508" layer="1"/>
 </signal>
 <signal name="VCC">
