File: Eagle/PhasedArray2/ADC_ADC7761BSTZ/ADC_AD7761BSTZ.sch (EAGLE design)
At the start: 42 parts, among them U1 AD7761BSTZ, Y1 HCM4932768000ABJT

Commit message: Add files via upload
Changed lines of the file:
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@@
 <segment>
 <pinref part="U1" gate="G$1" pin="MODE3/GPIO3"/>
-<wire x1="-45.7" y1="-17.8" x2="-45.7" y2="-17.78" width="0.1524" layer="91"/>
-<wire x1="-45.7" y1="-17.78" x2="-38.1" y2="-17.78" width="0.1524" layer="91"/>
 <pinref part="JP3" gate="A" pin="1"/>
-<wire x1="-45.7" y1="-17.78" x2="-58.06" y2="-17.78" width="0.1524" layer="91"/>
+<wire x1="-38.1" y1="-17.78" x2="-58.06" y2="-17.78" width="0.1524" layer="91"/>
 </segment>
 </net>

Commit message: Add files via upload
Parts:
- added S5, S6: CJS-1200TB, CJS-1200TB:CJS-1200TB
Connections:
- new net N$37: C21.1, S5.2, U1.REF1+
- new net VCC/2: C18.1, JP2.1, JP2.2, R4.2, S5.1, S6.1
- net N$36: now also C22.1, S6.2, U1.REF2+; no longer C18.1, JP2.1, JP2.2, R4.2
- net VCC: now also S5.3, S6.3; no longer C21.1, C22.1, U1.REF1+, U1.REF2+
Other:
- moved on the sheet: C21, C22
