File: Eagle/PhasedArray2/ADC_ADC7761BSTZ/ADC_AD7761BSTZ.brd (EAGLE design)
At the start: 100 x 80 mm, 42 parts, among them U1 AD7761BSTZ, Y1 HCM4932768000ABJT

Commit message: Add files via upload
Parts:
- moved C15 24.5 mm to (47.3, 24.4), turned to 180 degrees
- moved C1 21.1 mm to (22.7, 41.0), turned to 270 degrees
- moved R4 20.9 mm to (21.0, 46.7)
- moved C13 20.2 mm to (49.8, 13.4)
- moved C10 20.2 mm to (15.0, 32.3)
- moved C7 20.2 mm to (31.4, 37.1)
- moved C11 20.2 mm to (36.1, 19.0)
- moved C12 20.2 mm to (60.4, 25.0)
- moved C14 20.2 mm to (40.6, 13.2)
- moved C16 20.2 mm to (46.4, 10.8)
- moved C17 20.2 mm to (56.9, 21.9)
- moved C19 20.2 mm to (55.5, 10.5)
- moved C21 20.2 mm to (15.0, 30.0)
- moved C22 20.2 mm to (39.1, 30.0)
- moved C4 20.2 mm to (30.4, 39.3)
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Routing:
- net DGND: track 17.8 -> 60.4 mm, vias 0 -> 8
- net VDD: track 64.7 -> 98.2 mm, vias 2 -> 5
- net AGND: track 52.1 -> 75.3 mm, vias 0 -> 9
- net GND: track 22.5 -> 29.2 mm, vias 0 -> 3
- net N$5: track 17.2 -> 21.9 mm
- net N$7: track 23.1 -> 27.1 mm
- net N$26: track 9.91 -> 12.0 mm
- net N$33: track 13.7 -> 15.0 mm
- net N$36: track 18.1 -> 19.3 mm
- net VCC: track 169.0 -> 168.2 mm
- added copper zone on layer 16, net AGND
- added copper zone on layer 16, net DGND
- added copper zone on layer 16, net GND
Other:
- board size 100 x 80 mm -> 65 x 56 mm

Commit message: Add files via upload
Parts:
- added S5, S6: CJS-1200TB, CJS-1200TB:B-TYPE
- moved JP1 28.3 mm to (18.3, 56.3), turned to 0 degrees
- moved JP8 19.6 mm to (48.1, 56.4), turned to 180 degrees
- moved JP6 13.7 mm to (66.6, 14.2), turned to 270 degrees
- moved R3 13.0 mm to (41.6, 3.08)
- moved C15 11.9 mm to (58.7, 27.6), turned to 0 degrees
- moved R2 10.5 mm to (32.5, 36.1)
- moved C9 9.01 mm to (44.0, 21.0), turned to 270 degrees
- moved C7 8.81 mm to (40.1, 35.7)
- moved C20 7.96 mm to (60.4, 9.40), turned to 180 degrees
- moved JP7 7.96 mm to (13.8, 4.91), turned to 180 degrees
- moved R1 7.84 mm to (47.0, 20.6), turned to 270 degrees
- moved C10 7.83 mm to (21.9, 28.5), turned to 90 degrees
- moved S4 7.57 mm to (28.6, 44.0), turned to 270 degrees
- moved C5 7.52 mm to (42.7, 16.1), turned to 0 degrees
- moved S1 7.33 mm to (51.8, 20.8), turned to 180 degrees
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Connections:
- new net N$37: C21.1, S5.2, U1.6
- new net VCC/2: C18.1, JP2.1, JP2.2, R4.2, S5.1, S6.1
- net N$36: now also C22.1, S6.2, U1.43; no longer C18.1, JP2.1, JP2.2, R4.2
- net VCC: now also S5.3, S6.3; no longer C21.1, C22.1, U1.43, U1.6
Routing:
- net VDD: track 98.2 -> 34.6 mm, vias 5 -> 0
- net N$35: track 50.0 -> 0.00 mm
- net VCC: track 168.2 -> 126.9 mm
- net N$6: track 39.1 -> 0.00 mm, vias 1 -> 0
- net DGND: track 60.4 -> 23.5 mm, vias 8 -> 5
- net AIN3+: track 19.2 -> 49.7 mm
- net AIN3-: track 18.3 -> 48.0 mm
- net AIN7+: track 17.3 -> 46.8 mm
- net AIN2+: track 17.5 -> 46.8 mm
- net AIN2-: track 17.9 -> 46.3 mm
- net N$7: track 27.1 -> 0.00 mm
- net AIN7-: track 18.2 -> 45.0 mm
- net N$30: track 26.7 -> 0.00 mm
- net N$28: track 24.2 -> 0.00 mm
- net +9V: track 73.1 -> 49.6 mm
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Other:
- board size 65 x 56 mm -> 70 x 60 mm

Commit message: Add files via upload
Parts:
- moved R3 9.24 mm to (43.7, 12.1)
- moved R2 6.65 mm to (27.8, 40.9)
- moved C2 6.20 mm to (43.3, 3.49), turned to 90 degrees
- moved C16 3.90 mm to (53.3, 6.09)
- moved C3 3.29 mm to (43.2, 8.39), turned to 270 degrees
- moved C13 3.22 mm to (56.2, 10.2)
- moved JP3 3.00 mm to (3.36, 13.1)
- moved PS2 3.00 mm to (52.1, 10.8)
- moved S2 2.55 mm to (34.1, 41.5), turned to 180 degrees
- moved S4 2.08 mm to (27.9, 46.0), turned to 180 degrees
- moved Y1 2.00 mm to (38.0, 9.00), turned to 90 degrees
- moved S3 1.78 mm to (39.7, 45.8), turned to 180 degrees
- moved C5 1.41 mm to (43.7, 15.1)
- moved C9 1.30 mm to (43.9, 19.7)
- moved JP4 1.00 mm to (27.4, 3.81)
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Routing:
- net N$35: track 0.00 -> 51.4 mm
- net VCC/2: track 21.1 -> 68.4 mm, vias 2 -> 4
- net VDD: track 34.6 -> 78.5 mm, vias 0 -> 2
- net N$30: track 0.00 -> 34.3 mm, vias 0 -> 1
- net N$28: track 0.00 -> 33.4 mm, vias 0 -> 3
- net N$6: track 0.00 -> 33.1 mm, vias 0 -> 1
- net N$12: track 0.00 -> 29.3 mm
- net N$11: track 0.00 -> 28.4 mm
- net N$10: track 0.00 -> 27.6 mm
- net N$9: track 0.00 -> 26.8 mm
- net N$8: track 0.00 -> 26.0 mm
- net N$5: track 0.00 -> 21.5 mm
- net N$16: track 0.00 -> 20.4 mm
- net N$18: track 0.00 -> 19.6 mm
- net N$20: track 0.00 -> 19.0 mm
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